File: electronics/nanoRIghtAux/nanoRIghtAux.kicad_pcb (KiCad board)
At the start: 2 copper layers, 85.1 x 68.6 mm, 22 parts, among them J1 Conn_MM5451, J10 Conn_EA_GLCD, J11 Conn_MAX7219, J12 Conn_PWRInput, J13 Conn_MAX_Pwr, J2 Conn_HYDA, J3 Conn_HYDB, J4 Conn_FUEL_FR, J5 Conn_FUEL_AL, J6 Conn_MOT_D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

Commit message: Update nanoRIghtAux-B_Cu.gbr, nanoRIghtAux-Edge_Cuts.gbr, and 6 more files...
Parts:
- moved H2 100.4 mm to (139.7, 125.7)
- moved H3 100.4 mm to (217.2, 64.8)
- moved H4 1.80 mm to (217.2, 125.7)
- moved H1 0.93 mm to (139.7, 64.8)
Other:
- board text added: "RightAUX Controlboard"
- board text removed: "RightAUC Controlboard"
Changed lines of the file:
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@@
     )
-  )
-  (footprint "MountingHole:MountingHole_3.5mm" (layer "F.Cu")
-    (at 139.7 63.84)
-    (descr "Mounting Hole 3.5mm, no annular")
-    (tags "mounting hole 3.5mm no annular")
-    (property "Sheetfile" "nanoRIghtAux.kicad_sch")
-    (property "Sheetname" "")
-    (property "ki_description" "Mounting Hole without connection")
-    (property "ki_keywords" "mounting hole")
-    (attr exclude_from_pos_files)
-    (fp_text reference "H1" (at 0 -4.5) (layer "F.SilkS")
-        (effects (font (size 1 1) (thickness 0.15)))
-    )
-    (fp_text value "MountingHole" (at 0 4.5) (layer "F.Fab")
-        (effects (font (size 1 1) (thickness 0.15)))
-    )
-    (fp_text user "${REFERENCE}" (at 0 0) (layer "F.Fab")
-        (effects (font (size 1 1) (thickness 0.15)))
-    )
-    (fp_circle (center 0 0) (end 3.5 0)
-      (stroke (width 0.15) (type solid)) (fill none) (layer "Cmts.User"))
-    (fp_circle (center 0 0) (end 3.75 0)
-      (stroke (width 0.05) (type solid)) (fill none) (layer "F.CrtYd"))
-    (pad "" np_thru_hole circle (at 0 0) (size 3.5 3.5) (drill 3.5) (layers "*.Cu" "*.Mask"))
   )
   (footprint "Connector_PinHeader_2.54mm:PinHeader_1x04_P2.54mm_Vertical" (layer "F.Cu")
@@
       (rotate (xyz 0 0 0))
     )
+  )
+  (footprint "MountingHole:MountingHole_3.5mm" (layer "F.Cu")
+    (at 139.7 64.77)
+    (descr "Mounting Hole 3.5mm, no annular")
+    (tags "mounting hole 3.5mm no annular")
+    (property "Sheetfile" "nanoRIghtAux.kicad_sch")
+    (property "Sheetname" "")
+    (property "ki_description" "Mounting Hole without connection")
+    (property "ki_keywords" "mounting hole")
+    (attr exclude_from_pos_files)
+    (fp_text reference "H1" (at 0 -4.5) (layer "F.SilkS")
+        (effects (font (size 1 1) (thickness 0.15)))
+    )
+    (fp_text value "MountingHole" (at 0 4.5) (layer "F.Fab")
+        (effects (font (size 1 1) (thickness 0.15)))
+    )
+    (fp_text user "${REFERENCE}" (at 0 0) (layer "F.Fab")
+        (effects (font (size 1 1) (thickness 0.15)))
+    )
+    (fp_circle (center 0 0) (end 3.5 0)
+      (stroke (width 0.15) (type solid)) (fill none) (layer "Cmts.User"))
+    (fp_circle (center 0 0) (end 3.75 0)
+      (stroke (width 0.05) (type solid)) (fill none) (layer "F.CrtYd"))
+    (pad "" np_thru_hole circle (at 0 0) (size 3.5 3.5) (drill 3.5) (layers "*.Cu" "*.Mask"))
   )
   (footprint "Connector_PinSocket_2.54mm:PinSocket_1x03_P2.54mm_Vertical" (layer "F.Cu")
@@
       (rotate (xyz 0 0 0))
     )
-  )
-  (footprint "MountingHole:MountingHole_3.5mm" (layer "F.Cu")
-    (at 218.44 127)
-    (descr "Mounting Hole 3.5mm, no annular")
-    (tags "mounting hole 3.5mm no annular")
-    (property "Sheetfile" "nanoRIghtAux.kicad_sch")
-    (property "Sheetname" "")
-    (property "ki_description" "Mounting Hole without connection")
-    (property "ki_keywords" "mounting hole")
-    (attr exclude_from_pos_files)
-    (fp_text reference "H4" (at 0 -4.5) (layer "F.SilkS")
-        (effects (font (size 1 1) (thickness 0.15)))
-    )
-    (fp_text value "MountingHole" (at 0 4.5) (layer "F.Fab")
-        (effects (font (size 1 1) (thickness 0.15)))
-    )
-    (fp_text user "${REFERENCE}" (at 0 0) (layer "F.Fab")
-        (effects (font (size 1 1) (thickness 0.15)))
-    )
-    (fp_circle (center 0 0) (end 3.5 0)
-      (stroke (width 0.15) (type solid)) (fill none) (layer "Cmts.User"))
-    (fp_circle (center 0 0) (end 3.75 0)
-      (stroke (width 0.05) (type solid)) (fill none) (layer "F.CrtYd"))
-    (pad "" np_thru_hole circle (at 0 0) (size 3.5 3.5) (drill 3.5) (layers "*.Cu" "*.Mask"))
   )
   (footprint "Connector_PinHeader_2.54mm:PinHeader_1x04_P2.54mm_Vertical" (layer "F.Cu")
@@
   )
   (footprint "MountingHole:MountingHole_3.5mm" (layer "F.Cu")
-    (at 218.44 63.5)
+    (at 139.7 125.73)
     (descr "Mounting Hole 3.5mm, no annular")
     (tags "mounting hole 3.5mm no annular")
@@
     (attr exclude_from_pos_files)
     (fp_text reference "H2" (at 0 -4.5) (layer "F.SilkS")
-        (effects (font (size 1 1) (thickness 0.15)))
-    )
-    (fp_text value "MountingHole" (at 0 4.5) (layer "F.Fab")
-        (effects (font (size 1 1) (thickness 0.15)))
-    )
-    (fp_text user "${REFERENCE}" (at 0 0) (layer "F.Fab")
-        (effects (font (size 1 1) (thickness 0.15)))
-    )
-    (fp_circle (center 0 0) (end 3.5 0)
-      (stroke (width 0.15) (type solid)) (fill none) (layer "Cmts.User"))
-    (fp_circle (center 0 0) (end 3.75 0)
-      (stroke (width 0.05) (type solid)) (fill none) (layer "F.CrtYd"))
-    (pad "" np_thru_hole circle (at 0 0) (size 3.5 3.5) (drill 3.5) (layers "*.Cu" "*.Mask"))
-  )
-  (footprint "MountingHole:MountingHole_3.5mm" (layer "F.Cu")
-    (at 138.43 127)
-    (descr "Mounting Hole 3.5mm, no annular")
-    (tags "mounting hole 3.5mm no annular")
-    (property "Sheetfile" "nanoRIghtAux.kicad_sch")
-    (property "Sheetname" "")
-    (property "ki_description" "Mounting Hole without connection")
-    (property "ki_keywords" "mounting hole")
-    (attr exclude_from_pos_files)
-    (fp_text reference "H3" (at 0 -4.5) (layer "F.SilkS")
         (effects (font (size 1 1) (thickness 0.15)))
     )
@@
     )
   )
+  (footprint "MountingHole:MountingHole_3.5mm" (layer "F.Cu")
+    (at 217.17 64.77)
+    (descr "Mounting Hole 3.5mm, no annular")
+    (tags "mounting hole 3.5mm no annular")
+    (property "Sheetfile" "nanoRIghtAux.kicad_sch")
+    (property "Sheetname" "")
+    (property "ki_description" "Mounting Hole without connection")
+    (property "ki_keywords" "mounting hole")
+    (attr exclude_from_pos_files)
+    (fp_text reference "H3" (at 0 -4.5) (layer "F.SilkS")
+        (effects (font (size 1 1) (thickness 0.15)))
+    )
+    (fp_text value "MountingHole" (at 0 4.5) (layer "F.Fab")
+        (effects (font (size 1 1) (thickness 0.15)))
+    )
+    (fp_text user "${REFERENCE}" (at 0 0) (layer "F.Fab")
+        (effects (font (size 1 1) (thickness 0.15)))
+    )
+    (fp_circle (center 0 0) (end 3.5 0)
+      (stroke (width 0.15) (type solid)) (fill none) (layer "Cmts.User"))
+    (fp_circle (center 0 0) (end 3.75 0)
+      (stroke (width 0.05) (type solid)) (fill none) (layer "F.CrtYd"))
+    (pad "" np_thru_hole circle (at 0 0) (size 3.5 3.5) (drill 3.5) (layers "*.Cu" "*.Mask"))
+  )
   (footprint "Connector_PinHeader_2.54mm:PinHeader_2x03_P2.54mm_Vertical" (layer "F.Cu")
     (at 147.305 81.275 -90)
@@
     )
   )
+  (footprint "MountingHole:MountingHole_3.5mm" (layer "F.Cu")
+    (at 217.17 125.73)
+    (descr "Mounting Hole 3.5mm, no annular")
+    (tags "mounting hole 3.5mm no annular")
+    (property "Sheetfile" "nanoRIghtAux.kicad_sch")
+    (property "Sheetname" "")
+    (property "ki_description" "Mounting Hole without connection")
+    (property "ki_keywords" "mounting hole")
+    (attr exclude_from_pos_files)
+    (fp_text reference "H4" (at 0 -4.5) (layer "F.SilkS")
+        (effects (font (size 1 1) (thickness 0.15)))
+    )
+    (fp_text value "MountingHole" (at 0 4.5) (layer "F.Fab")
+        (effects (font (size 1 1) (thickness 0.15)))
+    )
+    (fp_text user "${REFERENCE}" (at 0 0) (layer "F.Fab")
+        (effects (font (size 1 1) (thickness 0.15)))
+    )
+    (fp_circle (center 0 0) (end 3.5 0)
+      (stroke (width 0.15) (type solid)) (fill none) (layer "Cmts.User"))
+    (fp_circle (center 0 0) (end 3.75 0)
+      (stroke (width 0.05) (type solid)) (fill none) (layer "F.CrtYd"))
+    (pad "" np_thru_hole circle (at 0 0) (size 3.5 3.5) (drill 3.5) (layers "*.Cu" "*.Mask"))
+  )
   (footprint "Connector_PinHeader_2.54mm:PinHeader_1x02_P2.54mm_Vertical" (layer "F.Cu")
     (at 151.13 123.19 90)
@@
     (effects (font (size 1.5 1.5) (thickness 0.3) bold) (justify left bottom))
   )
-  (gr_text "RightAUC Controlboard" (at 166.37 128.27) (layer "F.Cu")
+  (gr_text "RightAUX Controlboard" (at 166.37 128.27) (layer "F.Cu")
     (effects (font (size 2 2) (thickness 0.3) bold) (justify left bottom))
   )
